File: hard/InterfazSpectrum/esquema.brd (EAGLE design)
At the start: 100 x 50 mm, 17 parts, among them IC1 ATMEGA644-20PU, IC2 XC9572-PC44, IC3 LD1117, Q3 16 MHz, X1 ZX-EDGE

Commit message: Esquema: Añadido módulo wifi y conectores I/O
Parts:
- removed RESET_BTN: -, pinhead:1X03
- added IC4: ESP-07ESP-07, Esp-07:ESP-07
- added JP1: CPLD_PROG, pinhead:1X06
- added JP2: PROG/COMM, pinhead:1X04
- added LED1: (no value), led:LED3MM
- added R2, R4, R8: 1K, resistor:0207/10
- added R3, R5: 2K2, resistor:0207/10
- added R6, R7: 10K, resistor:0207/10
- added RESET: -, pinhead:1X03
- JP4: value PROG/COMM -> (none); device pinhead:1X04 -> pinhead:1X08
- JP5: value CPLD_PROG -> (none); device pinhead:1X06 -> pinhead:1X04
- moved JP5 80.0 mm to (82.5, 30.5), turned to 180 degrees
- moved JP4 45.5 mm to (87.6, 7.62), turned to 180 degrees
- moved R1 17.8 mm to (96.5, 35.6), turned to 90 degrees
- moved IC2 5.08 mm to (22.9, 26.7)
- moved C1 5.08 mm to (87.6, 47.0)
- moved C2 5.08 mm to (80.0, 47.0)
- moved Q3 5.08 mm to (83.8, 41.9)
- moved IC3 1.27 mm to (20.3, 43.2)
- moved C3 1.27 mm to (72.4, 29.2), turned to 180 degrees
- moved IC1 1.27 mm to (72.4, 19.1)
- renumbered JP6 to JP3
Connections:
- removed net RX2_5V: IC1.17
- new net CH_PH_PULLUP: IC4.3, R6.1
- new net GPIO15_PULLDOWN: IC4.10, R7.1
- new net N$1: IC4.15, R2.1, R3.2
- new net N$2: LED1.A, R8.2
- new net RST_WIFI_3.3V: IC4.1, R4.1, R5.2
- new net TX1_5V: IC1.17, R2.2
- net +3.3V: now also IC4.8, JP1.6, R6.2, R8.1; no longer JP5.6
- net +5V: now also JP2.3, R1.1; no longer JP4.3, R1.2
- net ANALOG0: now also JP4.1
- net ANALOG1: now also JP4.2
- net ANALOG2: now also JP4.3
- net ANALOG3: now also JP4.4
- net ANALOG4: now also JP4.5
- net ANALOG5: now also JP4.6
- net ANALOG6: now also JP4.7
- net ANALOG7: now also JP4.8
- net GND: now also IC4.9, JP1.5, JP2.4, R3.1, R5.1, R7.2, RESET.3; no longer JP4.4, JP5.5, RESET_BTN.3
- net IO4: now also JP5.1
- net IO5: now also JP5.2
- net IO6: now also JP5.3
- net IO7: now also JP5.4
- net LED1: now also LED1.K
- net RESET_UC: now also R1.2, RESET.1; no longer R1.1, RESET_BTN.1
- net RST_WIFI: now also R4.2
- net RX0_5V: now also JP2.2; no longer JP4.2
- net TCK: now also JP1.4; no longer JP5.4
- net TDI: now also JP1.2; no longer JP5.2
- net TDO: now also JP1.3; no longer JP5.3
- net TMS: now also JP1.1; no longer JP5.1
- net TX0_5V: now also JP2.1; no longer JP4.1
Routing:
- net N$2: track 40.6 -> 0.00 mm
Other:
- board text removed: "Modulo WiFi"

Commit message: Arregladas algunas señales que no estaban conectadas en el cpld, módulo wifi y conector edge.
Connections:
- removed net N$4: X1.A6
- removed net N$5: X1.A7
- net GND: now also X1.A6, X1.A7
- net RX1_5V: now also IC4.16
- net TDO: now also IC2.30
Changed lines of the file:
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@@
 <contactref element="C1" pad="1"/>
 <contactref element="C2" pad="1"/>
-<contactref element="IC1" pad="11"/>
 <contactref element="C3" pad="2"/>
 <contactref element="RESET" pad="3"/>
@@
 <contactref element="R5" pad="1"/>
 <contactref element="R7" pad="2"/>
+<contactref element="IC1" pad="11"/>
+<contactref element="X1" pad="A6"/>
+<contactref element="X1" pad="A7"/>
 <wire x1="86.36" y1="46.99" x2="92.71" y2="45.72" width="0" layer="19" extent="1-1"/>
 <wire x1="81.28" y1="46.99" x2="86.36" y2="46.99" width="0" layer="19" extent="1-1"/>
@@
 <wire x1="73.66" y1="11.43" x2="71.12" y2="26.67" width="0" layer="19" extent="1-1"/>
 <wire x1="48.26" y1="2.54" x2="73.66" y2="11.43" width="0" layer="19" extent="16-16"/>
-<wire x1="29.21" y1="22.86" x2="48.26" y2="2.54" width="0" layer="19" extent="16-16"/>
+<wire x1="30.48" y1="2.54" x2="48.26" y2="2.54" width="0" layer="19" extent="16-16"/>
+<wire x1="27.94" y1="2.54" x2="30.48" y2="2.54" width="0" layer="19" extent="16-16"/>
+<wire x1="29.21" y1="22.86" x2="30.48" y2="2.54" width="0" layer="19" extent="16-16"/>
 <wire x1="24.13" y1="33.02" x2="29.21" y2="22.86" width="0" layer="19" extent="1-1"/>
 <wire x1="20.32" y1="40.64" x2="24.13" y2="33.02" width="0" layer="19" extent="1-1"/>
@@
 <signal name="RX1_5V">
 <contactref element="IC1" pad="16"/>
+<contactref element="IC4" pad="16"/>
+<wire x1="55.26" y1="30.1" x2="58.42" y2="26.67" width="0" layer="19" extent="1-1"/>
 </signal>
 <signal name="TX1_5V">
@@
 <signal name="TDO">
 <contactref element="JP1" pad="3"/>
-</signal>
-<signal name="N$4">
-<contactref element="X1" pad="A6"/>
-</signal>
-<signal name="N$5">
-<contactref element="X1" pad="A7"/>
+<contactref element="IC2" pad="30"/>
+<wire x1="3.81" y1="33.02" x2="16.51" y2="33.02" width="0" layer="19" extent="1-1"/>
 </signal>
 <signal name="N$3">

Commit message: Modificada resistencia R8, el valor correcto es 300 Ohm
Parts:
- R8: value 1K -> 300
Changed lines of the file:
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@@
 <attribute name="SPICEPREFIX" value="R" x="68.58" y="38.1" size="1.778" layer="27" display="off"/>
 </element>
-<element name="R8" library="resistor" package="0207/10" value="1K" x="3.81" y="15.24" rot="R90">
+<element name="R8" library="resistor" package="0207/10" value="300" x="3.81" y="15.24" rot="R90">
 <attribute name="SPICEPREFIX" value="R" x="3.81" y="15.24" size="1.778" layer="27" rot="R90" display="off"/>
 </element>
